File: valrob-wb-soudure-1.kicad_pcb (KiCad board)
At the start: 2 copper layers, 85 x 50 mm, 36 parts, among them J1 Conn_01x03, J2 Conn_01x06, J3 Conn_01x02, J4 Conn_01x02, J5 Conn_01x02, J6 Conn_01x02, Q1 2N7000, SW1 SW_Push, SW2 SW_Push, SW3 SW_Push, SW4 SW_Push

Commit message: pcb: add valrobotik logo
Parts:
- added G*** (x3): LOGO, LOGO, B.Cu at (120.0, 107.6)
- moved G*** 24.8 mm to (110.0, 128.5)
